File: fabrication/arduino_nano_pcb(phase1)/arduino_nano_pcb(phase1).kicad_pcb (KiCad board)
At the start: 2 copper layers, 69.2 x 58 mm, 7 parts, among them J1 Conn_02x04_Odd_Even, J2 Conn_01x04_Pin

Commit message: feat(added_gerber): added gerber files for pcb mass production
Routing:
- net VCC: track 82.4 -> 84.9 mm
- net /MCU_TX_SENSOR_RX: track 19.1 -> 21.6 mm
- net /MCU_RX_SENSOR_TX: track 22.9 -> 25.4 mm
Changed lines of the file:
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@@
 			(plotframeref no)
 			(mode 1)
-			(useauxorigin no)
+			(useauxorigin yes)
 			(pdf_front_fp_property_popups yes)
 			(pdf_back_fp_property_popups yes)
@@
 			(sketchdnponfab yes)
 			(crossoutdnponfab yes)
-			(subtractmaskfromsilk no)
+			(subtractmaskfromsilk yes)
 			(outputformat 1)
 			(mirror no)
-			(drillshape 1)
+			(drillshape 0)
 			(scaleselection 1)
-			(outputdirectory "")
+			(outputdirectory "../arduino_nano_pcb(phase1)(gerber_files)/")
 		)
 	)
@@
 	(gr_rect
 		(start 44.5 75)
-		(end 52.5 81)
+		(end 51.5 81)
 		(stroke
 			(width 0.2)
@@
 		)
 		(fill no)
-		(layer "F.SilkS")
-	)
-	(gr_line
-		(start 55 67)
-		(end 98 67)
-		(stroke
-			(width 0.1)
-			(type dash)
-		)
-		(layer "F.SilkS")
-	)
-	(gr_line
-		(start 55 91)
-		(end 55 67)
-		(stroke
-			(width 0.1)
-			(type dash)
-		)
-		(layer "F.SilkS")
-	)
-	(gr_line
-		(start 57.42 78)
-		(end 55.5 77)
-		(stroke
-			(width 0.1)
-			(type default)
-		)
-		(layer "F.SilkS")
-	)
-	(gr_line
-		(start 95 67)
-		(end 95 91)
-		(stroke
-			(width 0.1)
-			(type dash)
-		)
-		(layer "F.SilkS")
-	)
-	(gr_line
-		(start 98 67)
-		(end 101 67)
-		(stroke
-			(width 0.1)
-			(type dash)
-		)
-		(layer "F.SilkS")
-	)
-	(gr_line
-		(start 98 91)
-		(end 55 91)
-		(stroke
-			(width 0.1)
-			(type dash)
-		)
-		(layer "F.SilkS")
-	)
-	(gr_line
-		(start 98 91)
-		(end 101 91)
-		(stroke
-			(width 0.1)
-			(type dash)
-		)
-		(layer "F.SilkS")
-	)
-	(gr_line
-		(start 101 67)
-		(end 101 91)
-		(stroke
-			(width 0.1)
-			(type dash)
-		)
 		(layer "F.SilkS")
 	)
@@
 	)
 	(gr_text "Sensor TX\nSensor RX\nGND\n+5V"
-		(at 48.5 78 0)
+		(at 48 78 0)
 		(layer "F.SilkS")
 		(effects
@@
 	)
 	(segment
+		(start 56.04 82)
+		(end 53.5 82)
+		(width 1.5)
+		(layer "B.Cu")
+		(net "VCC")
+	)
+	(segment
 		(start 101.5 80.27)
 		(end 101.070151 80.27)
@@
 	)
 	(segment
+		(start 56.04 74.38)
+		(end 53.5 74.38)
+		(width 1.5)
+		(layer "B.Cu")
+		(net "/MCU_RX_SENSOR_TX")
+	)
+	(segment
 		(start 61.64 81.317919)
 		(end 61.64 93)
@@
 		(start 57.242081 76.92)
 		(end 61.64 81.317919)
+		(width 1.5)
+		(layer "B.Cu")
+		(net "/MCU_TX_SENSOR_RX")
+	)
+	(segment
+		(start 56.04 76.92)
+		(end 53.5 76.92)
 		(width 1.5)
 		(layer "B.Cu")
@@
 		)
 	)
-	(group ""
-		(members "0e26a3cf-b54c-4482-aedd-3b9c7efbc5a5" "3aae7e45-8e1a-4678-808e-9a8f977607fc"
-			"4c92ca98-bffc-4cca-a9a0-f139ba0909fb" "58952a37-567e-4af5-ab70-0a5920670009"
-			"5c9683dd-0ab4-46e9-b4ea-2c14d77d01c7" "ca4601e6-ee34-4b01-b7c7-22fcc9bd6f74"
-			"f88167ee-ef8b-415a-bd00-8d8584c43847"
-		)
-	)
