File: fabrication/arduino_nano_pcb(phase1)/arduino_nano_pcb(phase1).kicad_sch (KiCad schematic)
At the start: 3 parts, among them J2 Conn_01x04_Pin, J3 Conn_01x04_Pin

Commit message: feat(added_pcb_phase_1): added pcb files for the phase 1 of the project that uses arduino nano
Parts:
- removed J3: Conn_01x04_Pin, symbol Connector:Conn_01x04_Pin
- added H1, H2, H3, H4: MountingHole_Pad, MountingHole:MountingHole_3.2mm_M3_Pad_TopBottom, symbol Mechanical:MountingHole_Pad
- added J1: Conn_02x04_Odd_Even, Connector_PinHeader_2.54mm:PinHeader_2x04_P2.54mm_Vertical, symbol Connector_Generic:Conn_02x04_Odd_Even
- J2: footprint (none) -> Connector_PinHeader_2.54mm:PinHeader_1x04_P2.54mm_Vertical
Connections:
- net GND: now also J2.4 (Pin_4), H1.1, H2.1, H3.1, H4.1, J1.5 (Pin_5), J1.6 (Pin_6)
- net VCC: now also J2.3 (Pin_3), J1.7 (Pin_7), J1.8 (Pin_8)
- net MCU_TX_SENSOR_RX: now reaches A1.15 (D12)
- net MCU_TX_SENSOR_RX: now also J1.3 (Pin_3), J1.4 (Pin_4)
- net TM1637_DIO: now reaches A1.5 (D2)
- net TM1637_DIO: now also J2.2 (Pin_2)
- net TM1637_CLK: now reaches A1.6 (D3)
- net TM1637_CLK: now also J2.1 (Pin_1)
- net Sensor_rx renamed MCU_RX_SENSOR_TX
- net MCU_RX_SENSOR_TX: now also J1.1 (Pin_1), J1.2 (Pin_2)
Other:
- note added: "GAS SENSOR INTERFACE"
- note added: "TM1637_DISPLAY"
- title: (none) -> DFRobot Multi-Gas Transmitter
- moved on the sheet: A1, J2

Commit message: feat(pcb_rev2): modified the pcb (rev 2)
Parts:
- removed J1: Conn_02x04_Odd_Even, Connector_PinHeader_2.54mm:PinHeader_2x04_P2.54mm_Vertical, symbol Connector_Generic:Conn_02x04_Odd_Even
- added J1: Conn_01x04_Pin, Connector_PinHeader_2.54mm:PinHeader_1x04_P2.54mm_Horizontal, symbol Connector:Conn_01x04_Pin
- H1: renamed from H4; footprint MountingHole:MountingHole_3.2mm_M3_Pad_TopBottom -> MountingHole:MountingHole_5mm_Pad_TopBottom
- H2: renamed from H3; footprint MountingHole:MountingHole_3.2mm_M3_Pad_TopBottom -> MountingHole:MountingHole_5mm_Pad_TopBottom
- H3: renamed from H2; footprint MountingHole:MountingHole_3.2mm_M3_Pad_TopBottom -> MountingHole:MountingHole_5mm_Pad_TopBottom
- H4: renamed from H1; footprint MountingHole:MountingHole_3.2mm_M3_Pad_TopBottom -> MountingHole:MountingHole_5mm_Pad_TopBottom
- J2: footprint Connector_PinHeader_2.54mm:PinHeader_1x04_P2.54mm_Vertical -> TM1637:TM1637
Connections:
- net GND: now also J1.3 (Pin_3)
- net MCU_RX_SENSOR_TX: now also J1.1 (Pin_1)
- net MCU_TX_SENSOR_RX: now also J1.2 (Pin_2)
- net VCC: now also J1.4 (Pin_4)
